File: kicad/keyboard.kicad_pcb (KiCad board)
At the start: 2 copper layers, 424.4 x 124.4 mm, 161 parts, among them SW1 SW_Push, SW10 SW_Push, SW11 SW_Push, SW12 SW_Push, SW13 SW_Push, SW14 SW_Push, SW15 SW_Push, SW16 SW_Push, SW17 SW_Push, SW18 SW_Push, SW19 SW_Push, SW2 SW_Push, SW20 SW_Push, SW21 SW_Push, SW22 SW_Push, SW23 SW_Push, SW24 SW_Push, SW25 SW_Push, SW26 SW_Push, SW27 SW_Push, SW28 SW_Push, SW29 SW_Push, SW3 SW_Push, SW30 SW_Push, SW31 SW_Push, SW32 SW_Push, SW33 SW_Push, SW34 SW_Push, SW35 SW_Push, SW36 SW_Push, SW37 SW_Push, SW38 SW_Push, SW39 SW_Push, SW4 SW_Push, SW40 SW_Push, SW41 SW_Push, SW42 SW_Push, SW43 SW_Push, SW44 SW_Push, SW45 SW_Push, SW46 SW_Push, SW47 SW_Push, SW48 SW_Push, SW49 SW_Push, SW5 SW_Push, SW50 SW_Push, SW51 SW_Push, SW52 SW_Push, SW53 SW_Push, SW54 SW_Push, SW55 SW_Push, SW56 SW_Push, SW57 SW_Push, SW58 SW_Push, SW59 SW_Push, SW6 SW_Push, SW60 SW_Push, SW61 SW_Push, SW62 SW_Push, SW63 SW_Push, SW64 SW_Push, SW65 SW_Push, SW66 SW_Push, SW67 SW_Push, SW68 SW_Push, SW69 SW_Push, SW7 SW_Push, SW70 SW_Push, SW71 SW_Push, SW72 SW_Push, SW73 SW_Push, SW74 SW_Push, SW75 SW_Push, SW76 SW_Push, SW77 SW_Push, SW78 SW_Push, SW79 SW_Push, SW8 SW_Push, SW80 SW_Push, SW9 SW_Push

Commit message: WIP
Connections:
- REF** pad 1: COL0 -> (no net)
- REF** pad 10: COL7 -> (no net)
- REF** pad 11: COL8 -> (no net)
- REF** pad 12: COL9 -> (no net)
- REF** pad 14: ROW0 -> (no net)
- REF** pad 15: ROW1 -> (no net)
- REF** pad 16: ROW2 -> (no net)
- REF** pad 2: COL1 -> (no net)
- REF** pad 21: COL12 -> ROW2
- REF** pad 22: COL13 -> ROW1
- REF** pad 24: COL14 -> ROW0
- REF** pad 25: COL15 -> (no net)
- REF** pad 26: COL16 -> (no net)
- REF** pad 27: COL17 -> (no net)
- REF** pad 29: COL18 -> (no net)
- REF** pad 31: COL19 -> (no net)
- REF** pad 32: COL20 -> (no net)
- REF** pad 34: COL21 -> (no net)
- REF** pad 4: COL2 -> (no net)
- REF** pad 5: COL3 -> (no net)
- REF** pad 6: COL4 -> (no net)
- REF** pad 7: COL5 -> (no net)
- REF** pad 9: COL6 -> (no net)
Routing:
- net COL21: track 215.8 -> 0.00 mm, vias 1 -> 0
- net COL0: track 229.9 -> 21.0 mm, vias 1 -> 0
- net COL1: track 272.5 -> 88.0 mm, vias 1 -> 0
- net COL20: track 246.6 -> 64.9 mm, vias 1 -> 0
- net COL2: track 255.1 -> 87.9 mm, vias 1 -> 0
- net COL19: track 253.3 -> 89.9 mm, vias 1 -> 0
- net COL3: track 215.7 -> 66.9 mm, vias 1 -> 0
- net COL18: track 236.0 -> 90.0 mm, vias 1 -> 0
- net COL17: track 196.9 -> 64.8 mm, vias 1 -> 0
- net COL4: track 196.9 -> 66.9 mm, vias 1 -> 0
- net COL16: track 188.8 -> 64.9 mm, vias 1 -> 0
- net COL5: track 201.5 -> 89.9 mm, vias 1 -> 0
- net COL14: track 215.7 -> 109.1 mm, vias 1 -> 0
- net COL8: track 100.0 -> 0.00 mm, vias 1 -> 0
- net COL15: track 207.7 -> 109.1 mm, vias 1 -> 0
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Other:
- copper layers 2 -> 4

Commit message: WIP
Connections:
- SW77 pad 1: COL10 -> COL9
Routing:
- net COL9: track 38.1 -> 89.0 mm

Commit message: WIP
Connections:
- REF** pad 1: (no net) -> COL0
- REF** pad 10: (no net) -> COL7
- REF** pad 11: (no net) -> COL8
- REF** pad 12: (no net) -> COL9
- REF** pad 14: (no net) -> ROW0
- REF** pad 15: (no net) -> ROW1
- REF** pad 16: (no net) -> ROW2
- REF** pad 2: (no net) -> COL1
- REF** pad 21: ROW2 -> COL12
- REF** pad 22: ROW1 -> COL13
- REF** pad 24: ROW0 -> COL14
- REF** pad 25: (no net) -> COL15
- REF** pad 26: (no net) -> COL16
- REF** pad 27: (no net) -> COL17
- REF** pad 29: (no net) -> COL18
- REF** pad 31: (no net) -> COL19
- REF** pad 32: (no net) -> COL20
- REF** pad 34: (no net) -> COL21
- REF** pad 4: (no net) -> COL2
- REF** pad 5: (no net) -> COL3
- REF** pad 6: (no net) -> COL4
- REF** pad 7: (no net) -> COL5
- REF** pad 9: (no net) -> COL6
Routing:
- net COL21: track 0.00 -> 215.5 mm, vias 0 -> 1
- net COL0: track 21.0 -> 232.5 mm, vias 0 -> 1
- net COL1: track 88.0 -> 270.4 mm, vias 0 -> 1
- net COL20: track 64.9 -> 247.0 mm, vias 0 -> 1
- net COL19: track 89.9 -> 253.6 mm, vias 0 -> 1
- net COL2: track 87.9 -> 250.7 mm, vias 0 -> 1
- net COL3: track 66.9 -> 210.6 mm, vias 0 -> 1
- net COL18: track 90.0 -> 231.2 mm, vias 0 -> 1
- net COL4: track 66.9 -> 190.3 mm, vias 0 -> 1
- net COL17: track 64.8 -> 180.3 mm, vias 0 -> 1
- net COL8: track 0.00 -> 107.9 mm, vias 0 -> 1
- net COL5: track 89.9 -> 193.1 mm, vias 0 -> 1
- net COL16: track 64.9 -> 162.2 mm, vias 0 -> 1
- net COL6: track 114.7 -> 199.0 mm, vias 0 -> 1
- net COL7: track 111.1 -> 190.5 mm, vias 0 -> 1
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Other:
- board text added: "Terminus Est"
- board text added: "made with love by @extremefraud art by @iamzoop thanks to @kh3dron && @dededecline"

Commit message: graphics
Parts:
- added G***: LOGO, LOGO, F.Cu at (344.1, 171.1)
- added G***: LOGO, LOGO, F.Cu at (249.1, 170.4)
- added G***: LOGO, LOGO, F.Cu at (296.0, 215.6)
- added REF**: MountingHole_2.1mm, MountingHole:MountingHole_2.1mm, F.Cu at (426.5, 218.8)
- added REF**: MountingHole_2.1mm, MountingHole:MountingHole_2.1mm, F.Cu at (351.0, 177.1)
- added REF**: MountingHole_2.1mm, MountingHole:MountingHole_2.1mm, F.Cu at (175.5, 237.5)
- added REF**: MountingHole_2.1mm, MountingHole:MountingHole_2.1mm, F.Cu at (506.5, 176.9)
- added REF**: MountingHole_2.1mm, MountingHole:MountingHole_2.1mm, F.Cu at (164.5, 218.6)
- added REF**: MountingHole_2.1mm, MountingHole:MountingHole_2.1mm, F.Cu at (334.5, 141.2)
- added REF**: MountingHole_2.1mm, MountingHole:MountingHole_2.1mm, F.Cu at (274.5, 237.2)
- added REF**: MountingHole_2.1mm, MountingHole:MountingHole_2.1mm, F.Cu at (237.6, 174.8)
- added REF**: MountingHole_2.1mm, MountingHole:MountingHole_2.1mm, F.Cu at (92.9, 149.6)
- added REF**: MountingHole_2.1mm, MountingHole:MountingHole_2.1mm, F.Cu at (499.8, 149.8)
- added REF**: MountingHole_2.1mm, MountingHole:MountingHole_2.1mm, F.Cu at (131.1, 234.5)
- added REF**: MountingHole_2.1mm, MountingHole:MountingHole_2.1mm, F.Cu at (311.9, 237.0)
- added REF**: MountingHole_2.1mm, MountingHole:MountingHole_2.1mm, F.Cu at (276.2, 192.4)
- added REF**: MountingHole_2.1mm, MountingHole:MountingHole_2.1mm, F.Cu at (412.5, 237.5)
- added REF**: MountingHole_2.1mm, MountingHole:MountingHole_2.1mm, F.Cu at (100.1, 199.9)
- added REF**: MountingHole_2.1mm, MountingHole:MountingHole_2.1mm, F.Cu at (106.9, 218.5)
- added REF**: MountingHole_2.1mm, MountingHole:MountingHole_2.1mm, F.Cu at (312.0, 192.2)
- added REF**: MountingHole_2.1mm, MountingHole:MountingHole_2.1mm, F.Cu at (91.5, 175.8)
- added REF**: MountingHole_2.1mm, MountingHole:MountingHole_2.1mm, F.Cu at (492.9, 199.8)

Commit message: WIP
Parts:
- removed the G*** at (249.1, 170.4)
- G***: moved to B.Cu
- moved G*** 49.2 mm to (295.7, 179.7), turned to 179 degrees

Commit message: WIP
Parts:
- moved REF** 163.2 mm to (262.5, 137.6)
- moved REF** 4.24 mm to (337.5, 138.2)
Routing:
- net COL2: track 250.7 -> 251.5 mm
