File: kicad/keyboard.kicad_pcb (KiCad board)
At the start: 4 copper layers, 424.4 x 124.4 mm, 182 parts, among them SW1 SW_Push, SW10 SW_Push, SW11 SW_Push, SW12 SW_Push, SW13 SW_Push, SW14 SW_Push, SW15 SW_Push, SW16 SW_Push, SW17 SW_Push, SW18 SW_Push, SW19 SW_Push, SW2 SW_Push, SW20 SW_Push, SW21 SW_Push, SW22 SW_Push, SW23 SW_Push, SW24 SW_Push, SW25 SW_Push, SW26 SW_Push, SW27 SW_Push, SW28 SW_Push, SW29 SW_Push, SW3 SW_Push, SW30 SW_Push, SW31 SW_Push, SW32 SW_Push, SW33 SW_Push, SW34 SW_Push, SW35 SW_Push, SW36 SW_Push, SW37 SW_Push, SW38 SW_Push, SW39 SW_Push, SW4 SW_Push, SW40 SW_Push, SW41 SW_Push, SW42 SW_Push, SW43 SW_Push, SW44 SW_Push, SW45 SW_Push, SW46 SW_Push, SW47 SW_Push, SW48 SW_Push, SW49 SW_Push, SW5 SW_Push, SW50 SW_Push, SW51 SW_Push, SW52 SW_Push, SW53 SW_Push, SW54 SW_Push, SW55 SW_Push, SW56 SW_Push, SW57 SW_Push, SW58 SW_Push, SW59 SW_Push, SW6 SW_Push, SW60 SW_Push, SW61 SW_Push, SW62 SW_Push, SW63 SW_Push, SW64 SW_Push, SW65 SW_Push, SW66 SW_Push, SW67 SW_Push, SW68 SW_Push, SW69 SW_Push, SW7 SW_Push, SW70 SW_Push, SW71 SW_Push, SW72 SW_Push, SW73 SW_Push, SW74 SW_Push, SW75 SW_Push, SW76 SW_Push, SW77 SW_Push, SW78 SW_Push, SW79 SW_Push, SW8 SW_Push, SW80 SW_Push, SW9 SW_Push

Commit message: WIP
Parts:
- moved REF** 5.49 mm to (501.8, 180.5)
- moved REF** 0.45 mm to (91.8, 175.6)
Routing:
- net COL9: track 129.2 -> 124.8 mm

Commit message: WIP
Parts:
- removed the REF** at (426.5, 218.8)
- removed the REF** at (351.0, 177.1)
- removed the REF** at (175.5, 237.5)
- removed the REF** at (501.8, 180.5)
- removed the REF** at (164.5, 218.6)
- removed the REF** at (337.5, 138.2)
- removed the REF** at (274.5, 237.2)
- removed the REF** at (237.6, 174.8)
- removed the REF** at (99.8, 150.8)
- removed the REF** at (496.2, 149.8)
- removed the REF** at (276.2, 192.4)
- removed the REF** at (311.9, 237.0)
- removed the REF** at (412.5, 237.5)
- removed the REF** at (262.5, 137.6)
- removed the REF** at (100.1, 199.9)
- removed the REF** at (106.9, 218.5)
- removed the REF** at (312.0, 192.2)
- removed the REF** at (91.8, 175.6)
- removed the REF** at (492.9, 199.8)
Routing:
- net COL9: track 124.8 -> 129.2 mm
Other:
- copper layers 4 -> 6

Commit message: WIP
Other:
- board size 424.4 x 124.4 mm -> 434 x 124.7 mm
- copper layers 6 -> 4

Commit message: wip
Parts:
- renumbered REF** to PICO
